Commit message: Update my_robot.urdf.xacro

File: my_robot_description/urdf/my_robot.urdf.xacro (robot description, xacro)
@@ -2,65 +2,156 @@
 <robot name="my_robot_arm" xmlns:xacro="http://www.ros.org/wiki/xacro">
   <xacro:property name="package_path" value="$(find my_robot_description)" />
-  <link name="world" />
-  <link name="base">
+  <link name="world"/>
+  <link name="base_link">
     <visual>
-      <origin xyz="0 0 0" rpy="0 0 0" />
+      <origin xyz="0 0 0" rpy="-1.5708 0 0"/>
       <geometry>
-        <mesh filename="${package_path}/meshes/base.stl" scale="0.001 0.001 0.001" />
+        <mesh filename="${package_path}/meshes/base_link.stl" scale="0.001 0.001 0.001"/>
       </geometry>
     </visual>
     <collision>
-      <origin xyz="0 0 0" rpy="0 0 0" />
+      <origin xyz="0 0 0" rpy="-1.5708 0 0"/>
       <geometry>
-        <mesh filename="${package_path}/meshes/base.stl" scale="0.001 0.001 0.001" />
+        <mesh filename="${package_path}/meshes/base_link.stl" scale="0.001 0.001 0.001"/>
       </geometry>
     </collision>
     <inertial>
-      <mass value="0.9" />
-      <inertia ixx="0.01" iyy="0.01" izz="0.01" ixy="0" ixz="0" iyz="0" />
+      <mass value="1.5"/>
+      <inertia ixx="0.01" ixy="0" ixz="0" iyy="0.01" iyz="0" izz="0.01"/>
     </inertial>
   </link>
-  <!-- <link name="base_link">
+  <link name="link_1_shoulder">
     <visual>
-      <origin xyz="0 0 0" rpy="0 0 0" />
       <geometry>
-        <mesh filename="${package_path}/meshes/base_link.stl" scale="0.001 0.001 0.001" />
+        <mesh filename="${package_path}/meshes/link_1_shoulder.stl" scale="0.001 0.001 0.001"/>
       </geometry>
     </visual>
     <collision>
-      <origin xyz="0 0 0" rpy="0 0 0" />
       <geometry>
-        <mesh filename="${package_path}/meshes/base_link.stl" scale="0.001 0.001 0.001" />
+        <mesh filename="${package_path}/meshes/link_1_shoulder.stl" scale="0.001 0.001 0.001"/>
       </geometry>
     </collision>
     <inertial>
-      <mass value="0.9" />
-      <inertia ixx="0.01" iyy="0.01" izz="0.01" ixy="0" ixz="0" iyz="0" />
+      <mass value="0.8"/>
+      <inertia ixx="0.01" ixy="0" ixz="0" iyy="0.01" iyz="0" izz="0.01"/>
     </inertial>
-  </link> -->
-  <joint name="world_to_base_fixed" type="fixed">
-    <parent link="world" />
-    <child link="base" />
-    <origin xyz="0 0 0" rpy="0 0 0" />
+  </link>
+  <link name="link_2_elbow">
+    <visual>
+      <geometry>
+        <mesh filename="${package_path}/meshes/link_2_elbow.stl" scale="0.001 0.001 0.001"/>
+      </geometry>
+    </visual>
+    <collision>
+      <geometry>
+        <mesh filename="${package_path}/meshes/link_2_elbow.stl" scale="0.001 0.001 0.001"/>
+      </geometry>
+    </collision>
+    <inertial>
+      <mass value="0.7"/>
+      <inertia ixx="0.01" ixy="0" ixz="0" iyy="0.01" iyz="0" izz="0.01"/>
+    </inertial>
+  </link>
+  <link name="link_3_wrist">
+    <visual>
+      <geometry>
+        <mesh filename="${package_path}/meshes/link_3_wrist.stl" scale="0.001 0.001 0.001"/>
+      </geometry>
+    </visual>
+    <collision>
+      <geometry>
+        <mesh filename="${package_path}/meshes/link_3_wrist.stl" scale="0.001 0.001 0.001"/>
+      </geometry>
+    </collision>
+    <inertial>
+      <mass value="0.5"/>
+      <inertia ixx="0.01" ixy="0" ixz="0" iyy="0.01" iyz="0" izz="0.01"/>
+    </inertial>
+  </link>
+  <link name="link_4_gripper">
+    <visual>
+      <geometry>
+        <mesh filename="${package_path}/meshes/link_4_gripper.stl" scale="0.001 0.001 0.001"/>
+      </geometry>
+    </visual>
+    <collision>
+      <geometry>
+        <mesh filename="${package_path}/meshes/link_4_gripper.stl" scale="0.001 0.001 0.001"/>
+      </geometry>
+    </collision>
+    <inertial>
+      <mass value="0.3"/>
+      <inertia ixx="0.01" ixy="0" ixz="0" iyy="0.01" iyz="0" izz="0.01"/>
+    </inertial>
+  </link>
+  <joint name="world_fixed" type="fixed">
+    <parent link="world"/>
+    <child link="base_link"/>
+    <origin xyz="0 0 0" rpy="0 0 0"/>
   </joint>
-  <!-- <joint name="turntable_joint" type="revolute">
-    <parent link="base" />
-    <child link="base_link" />
-    <origin xyz="0 0 0" rpy="0 0 0" />
-    <axis xyz="0 0 1" />
-    <limit lower="-3.14" upper="3.14" effort="10" velocity="1.0" />
-  </joint> -->
+  <joint name="joint_1_turntable" type="revolute">
+    <parent link="base_link"/>
+    <child link="link_1_shoulder"/>
+    <origin xyz="[X_FROM_CAD] [Y_FROM_CAD] [Z_FROM_CAD]" rpy="0 0 0"/>
+    <axis xyz="0 0 1"/>
+    <limit lower="-3.14" upper="3.14" effort="10" velocity="1"/>
+  </joint>
+  <joint name="joint_2_shoulder" type="revolute">
+    <parent link="link_1_shoulder"/>
+    <child link="link_2_elbow"/>
+    <origin xyz="[X_FROM_CAD] [Y_FROM_CAD] [Z_FROM_CAD]" rpy="0 0 0"/>
+    <axis xyz="0 1 0"/>
+    <limit lower="-1.57" upper="1.57" effort="10" velocity="1"/>
+  </joint>
+  <joint name="joint_3_elbow" type="revolute">
+    <parent link="link_2_elbow"/>
+    <child link="link_3_wrist"/>
+    <origin xyz="[X_FROM_CAD] [Y_FROM_CAD] [Z_FROM_CAD]" rpy="0 0 0"/>
+    <axis xyz="0 1 0"/>
+    <limit lower="-1.57" upper="1.57" effort="10" velocity="1"/>
+  </joint>
+  <joint name="joint_4_wrist_pitch" type="revolute">
+    <parent link="link_3_wrist"/>
+    <child link="link_4_gripper"/>
+    <origin xyz="[X_FROM_CAD] [Y_FROM_CAD] [Z_FROM_CAD]" rpy="0 0 0"/>
+    <axis xyz="0 1 0"/>
+    <limit lower="-1.57" upper="1.57" effort="10" velocity="1"/>
+  </joint>
   <ros2_control name="GazeboSystem" type="system">
     <hardware>
       <plugin>gazebo_ros2_control/GazeboSystem</plugin>
     </hardware>
-    <!-- <joint name="turntable_joint">
+    <joint name="joint_1_turntable">
       <command_interface name="position">
         <param name="min">-3.14</param>
         <param name="max">3.14</param>
       </command_interface>
-      <state_interface name="position" />
-      <state_interface name="velocity" />
-    </joint> -->
+      <state_interface name="position"/>
+      <state_interface name="velocity"/>
+    </joint>
+    <joint name="joint_2_shoulder">
+      <command_interface name="position">
+        <param name="min">-1.57</param>
+        <param name="max">1.57</param>
+      </command_interface>
+      <state_interface name="position"/>
+      <state_interface name="velocity"/>
+    </joint>
+    <joint name="joint_3_elbow">
+      <command_interface name="position">
+        <param name="min">-1.57</param>
+        <param name="max">1.57</param>
+      </command_interface>
+      <state_interface name="position"/>
+      <state_interface name="velocity"/>
+    </joint>
+    <joint name="joint_4_wrist_pitch">
+      <command_interface name="position">
+        <param name="min">-1.57</param>
+        <param name="max">1.57</param>
+      </command_interface>
+      <state_interface name="position"/>
+      <state_interface name="velocity"/>
+    </joint>
   </ros2_control>
 </robot>
